File: ALRON-1600.kicad_sch (KiCad schematic)
At the start: 69 parts

Commit message: Add files via upload
Parts:
- removed R?: 4k7, symbol Device:R
- added D1, D2, D3, D4, D5: D, symbol Device:D
- added R1: 4k7, symbol Device:R
- added R2: 470k, symbol Device:R
- R?: value 4k6 -> 4k7
Connections:
- net +IN1: now also D5.2 (A)
- net +IN2: now also R2.2
- net GND: now also D4.2 (A)
- net OPAMP2-V+: now also D4.1 (K), D5.1 (K), R2.1
- net at C?.2, J?.2 (Pin_2): now also R1.2
- net at C?.2, Q?.3 (B), Q?.3 (C): now also D3.2 (A)
- net at Q?.3 (B): now also D1.1 (K), R1.1
- new net: D2.2 (A), D3.1 (K)
- new net: D1.2 (A), D2.1 (K)
Other:
- moved on the sheet: C?, J?, R?
